File: hardware/ssr_12v_by4/ssr_12v_by4.kicad_pcb (KiCad board)
At the start: 2 copper layers, 65 x 90 mm, 50 parts, among them J1 1190297, J2 1190297, J3 1190297, J4 1190297, Q1 IRF4905PBF, Q2 IRF4905PBF, Q3 IRF4905PBF, Q4 IRF4905PBF

Commit message: Part 1 of 'Never To Much Silkscreen'
Other:
- board text added: "Licensed under CERN-OHL-W v2"
- board text added: "v0.0.8"
- board text removed: "v0.0.3"
Changed lines of the file:
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@@
   (title_block
     (title "Solid State Relays 12 Volt x4")
-    (date "2022-12-31")
-    (rev "0.0.3")
+    (date "2023-01-03")
+    (rev "0.0.8")
     (comment 2 "creativecommons.org/licenses/by/4.0/")
     (comment 3 "License: CC By 4.0")
@@
     (effects (font (size 1 1) (thickness 0.15)) (justify mirror))
   )
+  (gr_text "Licensed under CERN-OHL-W v2" (at 85.5 95) (layer "F.SilkS")
+    (effects (font (size 1 1) (thickness 0.15)))
+  )
   (gr_text "+BATT\n a1\n a2\n a3\n a4" (at 109.65 70.9) (layer "F.SilkS")
     (effects (font (size 1 1) (thickness 0.15)) (justify left))
   )
-  (gr_text "© 2022 Michael Cummings" (at 85 94.5) (layer "F.SilkS")
+  (gr_text "© 2022 Michael Cummings" (at 85 93.5) (layer "F.SilkS")
     (effects (font (size 1 1) (thickness 0.15)))
   )
@@
     (effects (font (size 1.5 1.5) (thickness 0.2)))
   )
-  (gr_text "v0.0.3" (at 51 127.5) (layer "F.SilkS")
+  (gr_text "v0.0.8" (at 51 127.5) (layer "F.SilkS")
     (effects (font (size 1.5 1.5) (thickness 0.25)) (justify left))
   )
